Commit message: add eyes to dog

File: Task5/ex05/my_dog_robot/my_dog_robot/description/dog_with_cap.urdf (robot description, URDF)
Before this commit: robot dog, 18 links, 17 joints
Links:
- added link left_eye; visual sphere radius=0.01
- added link right_eye; visual sphere radius=0.01
Joints:
- added joint toleft_eye: type fixed, parent head, child left_eye, origin xyz=0.101 0.05 0.02
- added joint toright_eye: type fixed, parent head, child right_eye, origin xyz=0.101 -0.05 0.02
